File: 8x8_Matrix.kicad_sch (KiCad schematic)
At the start: 66 parts, among them J2 Conn_01x03

Commit message: Finished PCB front
Parts:
- J1: value (none) -> Conn_01x03
Changed lines of the file:
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@@
       (effects (font (size 1.27 1.27)) hide)
     )
-    (property "Value" "" (id 1) (at 62.23 261.62 0))
+    (property "Value" "+5V" (id 1) (at 62.23 261.62 0))
     (property "Footprint" "" (id 2) (at 62.23 266.7 0)
       (effects (font (size 1.27 1.27)) hide)
@@
       (effects (font (size 1.27 1.27)) hide)
     )
-    (property "Value" "" (id 1) (at 55.88 44.45 0)
+    (property "Value" "GND" (id 1) (at 55.88 44.45 0)
       (effects (font (size 1.27 1.27)) (justify left))
     )
@@
       (effects (font (size 1.27 1.27)) hide)
     )
-    (property "Value" "" (id 1) (at 54.61 26.67 0)
+    (property "Value" "+5V" (id 1) (at 54.61 26.67 0)
       (effects (font (size 1.27 1.27)) (justify left))
     )
@@
       (effects (font (size 1.27 1.27)) (justify left))
     )
-    (property "Value" "" (id 1) (at 38.1 270.5099 0)
+    (property "Value" "Conn_01x03" (id 1) (at 38.1 270.5099 0)
       (effects (font (size 1.27 1.27)) (justify left))
     )
@@
       (effects (font (size 1.27 1.27)) hide)
     )
-    (property "Value" "" (id 1) (at 62.23 276.86 0))
+    (property "Value" "GND" (id 1) (at 62.23 276.86 0))
     (property "Footprint" "" (id 2) (at 62.23 271.78 0)
       (effects (font (size 1.27 1.27)) hide)

Commit message: Finished PCB Back
Parts:
- D1: value (none) -> SK6805; footprint (none) -> LED_SMD:LED_SK6812_EC15_1.5x1.5mm
- J1: value Conn_01x03 -> (none)
Changed lines of the file:
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@@
     (in_bom yes) (on_board yes)
     (property "Reference" "D1" (id 0) (at 53.34 21.59 0))
-    (property "Value" "" (id 1) (at 53.34 24.13 0))
-    (property "Footprint" "" (id 2) (at 54.61 43.18 0)
+    (property "Value" "SK6805" (id 1) (at 53.34 24.13 0))
+    (property "Footprint" "LED_SMD:LED_SK6812_EC15_1.5x1.5mm" (id 2) (at 54.61 43.18 0)
       (effects (font (size 1.27 1.27)) (justify left top) hide)
     )
@@
       (effects (font (size 1.27 1.27)) (justify left))
     )
-    (property "Value" "Conn_01x03" (id 1) (at 38.1 270.5099 0)
-      (effects (font (size 1.27 1.27)) (justify left))
-    )
+    (property "Value" "" (id 1) (at 38.1 270.5099 0)
+      (effects (font (size 1.27 1.27)) (justify left))
+    )
