File: SK6805EC15_Matrix.kicad_pcb (KiCad board)
At the start: 2 copper layers, 20 x 20 mm, 70 parts

Commit message: Fixed typo
Parts:
- ?: footprint easyeda:PADPAD -> (none)
Changed lines of the file:
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@@
     )
   )
-  (footprint "easyeda:PADPAD" (layer "F.Cu")
+  (footprint "" (layer "F.Cu")
     (at 132.5 94.23)
-    (attr smd)
-    (fp_text reference "" (at 0.001 -0.253) (layer "B.SilkS") hide
-      (effects (font (size 1.143 1.143) (thickness 0.152)) (justify left mirror))
+    (fp_text reference "" (at 0.001 -0.253) (layer "F.SilkS")
+      (effects (font (size 1.143 1.143) (thickness 0.152)) (justify left))
     )
-    (fp_text value "" (at 0.001 -2.031) (layer "B.Fab") hide
-      (effects (font (size 1.143 1.143) (thickness 0.152)) (justify left mirror))
-    )
-    (fp_text user "ggeef5b64397d4c374c" (at 0 0) (layer "Cmts.User")
-      (effects (font (size 1 1) (thickness 0.15)))
+    (fp_text value "" (at 0.001 -2.031) (layer "F.SilkS")
+      (effects (font (size 1.143 1.143) (thickness 0.152)) (justify left))
     )
     (pad "1" smd rect (at 0 1.27) (size 5.08 2.54) (layers "B.Cu" "B.Paste" "B.Mask")
